Commit message: Tue Mar 19 00:52:43 CST 2019 successfully spawn two camera with correct tfpre and ns but lack of tf between two tf tree

File: camera_description/robots/camera.urdf.xacro (robot description, xacro)
@@ -1,11 +1,19 @@
 <?xml version="1.0"?>
-<robot name="ironfish" xmlns:xacro="http://www.ros.org/wiki/xacro">
-  <!-- Base and wheel for ironfish -->
+<robot name="desk_camera" xmlns:xacro="http://www.ros.org/wiki/xacro">
+  <xacro:arg name="nsp" default="c0" />
+  <xacro:arg name="tfpre" default="c0_tf" />
+  <!-- Base -->
   <xacro:include filename="$(find camera_description)/urdf/base/base.urdf.xacro"/>
-  <!-- colors for ironfish -->
+  <!-- camera -->
+  <xacro:include filename="$(find camera_description)/urdf/sensors/_d435.urdf.xacro"/>
+  <!-- colors  -->
   <xacro:include filename="$(find camera_description)/urdf/materials.xacro"/>
   <!-- Variables -->
   <xacro:property name="M_PI" value="3.1415926535897931" />
-  <!-- Use the macros to define ironfish -->
-  <xacro:camera_base/>
+  <!-- base -->
+  <xacro:camera_base name="deskCam" nsp="$(arg nsp)" tfpre="$(arg tfpre)"/>
+  <!-- Intel realsense-->
+  <xacro:sensor_d435 name="camera" parent="deskCam_base_link" nsp="$(arg nsp)" tfpre="$(arg tfpre)">
+    <origin xyz="0.0 0.0 0.0" rpy="0 0 0"/>
+  </xacro:sensor_d435>
 </robot>

File: camera_description/urdf/base/base.gazebo.xacro (robot description, xacro)
@@ -3,6 +3,6 @@
 <robot xmlns:xacro="http://ros.org/wiki/xacro">
   <!-- Base -->
-  <xacro:macro name="camera_base_gazebo">
-    <gazebo reference="desk_camera_base_link">
+  <xacro:macro name="camera_base_gazebo" params="name nsp tfpre">
+    <gazebo reference="${tfpre}/${name}_base_link">
       <material>Gazebo/White</material>
       <mu1 value="0.0"/>

File: camera_description/urdf/base/base.urdf.xacro (robot description, xacro)
@@ -2,8 +2,7 @@
 <robot xmlns:xacro="http://www.ros.org/wiki/xacro">
   <xacro:include filename="$(find camera_description)/urdf/base/base.gazebo.xacro" />
-  <xacro:include filename="$(find camera_description)/urdf/sensors/_d435.urdf.xacro" />
   <xacro:property name="pi" value="3.1415926535897931" />
-  <xacro:macro name="camera_base">
-      <link name="desk_camera_base_link">
+  <xacro:macro name="camera_base" params="name nsp tfpre">
+      <link name="${name}_base_link">
         <inertial>
           <origin
@@ -38,10 +37,6 @@
         </collision>
       </link>
-    <!-- Intel realsense-->
-    <sensor_d435 parent="desk_camera_base_link">
-      <origin xyz="0.0 0.0 0.0" rpy="0 0 0"/>
-    </sensor_d435>
     <!-- Extensions -->
-    <xacro:camera_base_gazebo/>
+    <xacro:camera_base_gazebo name="${name}" nsp="${nsp}" tfpre="${tfpre}"/>
   </xacro:macro>
 </robot>

File: camera_description/urdf/sensors/_d435.gazebo.xacro (robot description, xacro)
@@ -3,5 +3,7 @@
   <xacro:property name="M_PI" value="3.1415926535897931" />
   <!-- d435 camera for simulation -->
-  <xacro:macro name="_d435_gazebo" params="name">
+  <!--note that the namespace and tfpre are already processed behind-->
+  <!--DONT manually add the nsp or tfpre before each topics and frames-->
+  <xacro:macro name="_d435_gazebo" params="name nsp tfpre">
     <gazebo reference="${name}_depth_frame">
       <sensor type="depth" name="${name}">
@@ -19,5 +21,5 @@
           </clip>
         </camera>
-        <plugin name="${name}_camera_controller" filename="libgazebo_ros_openni_kinect.so">
+        <plugin name="camera_controller" filename="libgazebo_ros_openni_kinect.so">
           <alwaysOn>true</alwaysOn>
           <updateRate>20</updateRate>

File: camera_description/urdf/sensors/_d435.urdf.xacro (robot description, xacro)
@@ -6,7 +6,7 @@
 aluminum peripherial evaluation case.
 -->
-<robot xmlns:xacro="http://ros.org/wiki/xacro">
-  <xacro:include filename="$(find camera_description)/urdf/sensors/_d435.gazebo.xacro"/>
-  <xacro:macro name="sensor_d435" params="parent *origin">
+<robot name="sensor_d435" xmlns:xacro="http://ros.org/wiki/xacro">
+  <xacro:include filename="$(find camera_description)/urdf/sensors/_d435.gazebo.xacro" />
+  <xacro:macro name="sensor_d435" params="parent *origin name nsp tfpre">
     <xacro:property name="M_PI" value="3.1415926535897931" />
     <!-- The following values are approximate, and the camera node
@@ -31,15 +31,15 @@
     </material>
     <!-- camera body, with origin at bottom screw mount -->
-    <joint name="desk_camera_joint" type="fixed">
+    <joint name="camera_joint" type="fixed">
       <xacro:insert_block name="origin" />
       <parent link="${parent}"/>
-      <child link="desk_camera_link" />
+      <child link="camera_link" />
     </joint>
-    <link name="desk_camera_link">
+    <link name="camera_link">
       <visual>
       <origin xyz="${d435_cam_mount_from_center_offset} 0.0 ${d435_cam_height/2}" rpy="${M_PI/2} 0 ${M_PI/2}"/>
         <geometry>
           <!-- <box size="${d435_cam_width} ${d435_cam_height} ${d435_cam_depth}"/> -->
-	  <mesh filename="package://camera_description/meshes/intel_realsense_d435/d435.dae" />
+	  <mesh filename="package://realsense2_camera/meshes/d435.dae" />
           <!--<mesh filename="package://realsense2_camera/meshes/d435/d435.dae" />-->
         </geometry>
@@ -60,57 +60,57 @@
     </link>
     <!-- camera depth joints and links -->
-    <joint name="desk_camera_depth_joint" type="fixed">
+    <joint name="camera_depth_joint" type="fixed">
       <origin xyz="${d435_cam_depth_px} ${d435_cam_depth_py} ${d435_cam_depth_pz}" rpy="0 0 0"/>
-      <parent link="desk_camera_link"/>
-      <child link="desk_camera_depth_frame" />
+      <parent link="camera_link"/>
+      <child link="camera_depth_frame" />
     </joint>
-    <link name="desk_camera_depth_frame"/>
-    <joint name="desk_camera_depth_optical_joint" type="fixed">
+    <link name="camera_depth_frame"/>
+    <joint name="camera_depth_optical_joint" type="fixed">
       <origin xyz="0 0 0" rpy="${-M_PI/2} 0 ${-M_PI/2}" />
-      <parent link="desk_camera_depth_frame" />
-      <child link="desk_camera_depth_optical_frame" />
+      <parent link="camera_depth_frame" />
+      <child link="camera_depth_optical_frame" />
     </joint>
-    <link name="desk_camera_depth_optical_frame"/>
+    <link name="camera_depth_optical_frame"/>
     <!-- camera left IR joints and links -->
-    <joint name="desk_camera_left_ir_joint" type="fixed">
+    <joint name="camera_left_ir_joint" type="fixed">
       <origin xyz="0 ${d435_cam_depth_to_left_ir_offset} 0" rpy="0 0 0" />
-      <parent link="desk_camera_depth_frame" />
-      <child link="desk_camera_left_ir_frame" />
+      <parent link="camera_depth_frame" />
+      <child link="camera_left_ir_frame" />
     </joint>
-    <link name="desk_camera_left_ir_frame"/>
-    <joint name="desk_camera_left_ir_optical_joint" type="fixed">
+    <link name="camera_left_ir_frame"/>
+    <joint name="camera_left_ir_optical_joint" type="fixed">
       <origin xyz="0 0 0" rpy="${-M_PI/2} 0 ${-M_PI/2}" />
-      <parent link="desk_camera_left_ir_frame" />
-      <child link="desk_camera_left_ir_optical_frame" />
+      <parent link="camera_left_ir_frame" />
+      <child link="camera_left_ir_optical_frame" />
     </joint>
-    <link name="desk_camera_left_ir_optical_frame"/>
-    <!-- desk_camera right IR joints and links -->
-    <joint name="desk_camera_right_ir_joint" type="fixed">
+    <link name="camera_left_ir_optical_frame"/>
+    <!-- camera right IR joints and links -->
+    <joint name="camera_right_ir_joint" type="fixed">
       <origin xyz="0 ${d435_cam_depth_to_right_ir_offset} 0" rpy="0 0 0" />
-      <parent link="desk_camera_depth_frame" />
-      <child link="desk_camera_right_ir_frame" />
+      <parent link="camera_depth_frame" />
+      <child link="camera_right_ir_frame" />
     </joint>
-    <link name="desk_camera_right_ir_frame"/>
-    <joint name="desk_camera_right_ir_optical_joint" type="fixed">
+    <link name="camera_right_ir_frame"/>
+    <joint name="camera_right_ir_optical_joint" type="fixed">
       <origin xyz="0 0 0" rpy="${-M_PI/2} 0 ${-M_PI/2}" />
-      <parent link="desk_camera_right_ir_frame" />
-      <child link="desk_camera_right_ir_optical_frame" />
+      <parent link="camera_right_ir_frame" />
+      <child link="camera_right_ir_optical_frame" />
     </joint>
-    <link name="desk_camera_right_ir_optical_frame"/>
-    <!-- desk_camera color joints and links -->
-    <joint name="desk_camera_color_joint" type="fixed">
+    <link name="camera_right_ir_optical_frame"/>
+    <!-- camera color joints and links -->
+    <joint name="camera_color_joint" type="fixed">
       <origin xyz="0 ${d435_cam_depth_to_color_offset} 0" rpy="0 0 0" />
-      <parent link="desk_camera_depth_frame" />
-      <child link="desk_camera_color_frame" />
+      <parent link="camera_depth_frame" />
+      <child link="camera_color_frame" />
     </joint>
-    <link name="desk_camera_color_frame"/>
-    <joint name="desk_camera_color_optical_joint" type="fixed">
+    <link name="camera_color_frame"/>
+    <joint name="camera_color_optical_joint" type="fixed">
       <origin xyz="0 0 0" rpy="${-M_PI/2} 0 ${-M_PI/2}" />
-      <parent link="desk_camera_color_frame" />
-      <child link="desk_camera_color_optical_frame" />
+      <parent link="camera_color_frame" />
+      <child link="camera_color_optical_frame" />
     </joint>
-    <link name="desk_camera_color_optical_frame"/>
+    <link name="camera_color_optical_frame"/>
     <!-- extensions -->
-    <xacro:_d435_gazebo name="desk_camera"/>
+    <xacro:_d435_gazebo name="${name}" nsp="${nsp}" tfpre="${tfpre}"/>
   </xacro:macro>
 </robot>
