Commit message: Sun Mar 24 01:33:03 CST 2019 create tf broadcaster to connect odom to camera_base_link

File: desk_description/urdf/base/base.urdf.xacro (robot description, xacro)
@@ -5,35 +5,11 @@
   <xacro:macro name="camera_base" params="name nsp tfpre">
       <link name="${name}_base_link">
-        <inertial>
-          <origin
-            xyz="0.0 0.0 0.0"
-            rpy="0 0 0" />
-          <mass
-            value="99.63917377366023" />
-          <inertia
-            ixx="0.23820634587875"
-            ixy="0"
-            ixz="0"
-            iyy="0.23820634587875"
-            iyz="0"
-            izz="0.23820634587875" />
-        </inertial>
-        <visual>
-          <origin
-            xyz="0 0 0"
-            rpy="0 0 0" />
-          <geometry>
-            <!--box size="10 10 10"/-->
-          </geometry>
-          <material name="white"/>
-        </visual>
-        <collision>
-          <origin
-            xyz="0 0 0"
-            rpy="0 0 0" />
-          <geometry>
-            <!--box size="10 10 10"/-->
-          </geometry>
-        </collision>
+            <visual>
+              <origin xyz="0 0 0" rpy="0 0 0"/>
+              <geometry>
+                <box size="0.01 0.01 0.01" />
+              </geometry>
+              <material name="White" />
+            </visual>
       </link>
     <!-- Extensions -->
